File: switching-circuit.kicad_sch (KiCad schematic)
At the start: 10 parts, among them Q1 2N3904, Q2 2N3904

Commit message: added power supply schematic, and deleted the -backups folder
Changed lines of the file:
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@@
   (junction (at 207.01 87.63) (diameter 0) (color 0 0 0 0)
   )
-  (junction (at 218.44 87.63) (diameter 0) (color 0 0 0 0)
-  )
   (wire (pts (xy 207.01 77.47) (xy 207.01 87.63))
     (stroke (width 0) (type default))
@@
     (stroke (width 0) (type default))
   )
-  (wire (pts (xy 218.44 85.09) (xy 218.44 87.63))
-    (stroke (width 0) (type default))
-  )
-  (wire (pts (xy 207.01 87.63) (xy 218.44 87.63))
-    (stroke (width 0) (type default))
-  )
   (wire (pts (xy 180.34 97.79) (xy 180.34 100.33))
     (stroke (width 0) (type default))
@@
     (stroke (width 0) (type default))
   )
-  (wire (pts (xy 218.44 87.63) (xy 220.98 87.63))
+  (wire (pts (xy 207.01 87.63) (xy 220.98 87.63))
     (stroke (width 0) (type default))
   )
@@
   (wire (pts (xy 207.01 100.33) (xy 200.66 100.33))
     (stroke (width 0) (type default))
+  )
+  (global_label "+5V" (shape input) (at 220.98 87.63 0) (fields_autoplaced)
+    (effects (font (size 1.27 1.27)) (justify left))
+    (property "Intersheetrefs" "${INTERSHEET_REFS}" (at 227.1021 87.63 0)
+      (effects (font (size 1.27 1.27)) (justify left) hide)
+    )
   )
   (global_label "S0" (shape input) (at 180.34 97.79 90) (fields_autoplaced)
@@
         )
       )
-    )
-  )
-  (symbol (lib_id "power:PWR_FLAG") (at 218.44 85.09 0) (unit 1)
-    (in_bom yes) (on_board yes) (dnp no) (fields_autoplaced)
-    (property "Reference" "#FLG02" (at 218.44 83.185 0)
-      (effects (font (size 1.27 1.27)) hide)
-    )
-    (property "Value" "PWR_FLAG" (at 218.44 80.01 0)
-      (effects (font (size 1.27 1.27)))
-    )
-    (property "Footprint" "" (at 218.44 85.09 0)
-      (effects (font (size 1.27 1.27)) hide)
-    )
-    (property "Datasheet" "~" (at 218.44 85.09 0)
-      (effects (font (size 1.27 1.27)) hide)
-    )
-    (pin "1")
-    (instances
-      (project "switched-bandpass-filter"
-        (path "/05f50450-de9a-44de-96d4-4a146d783d83"
-          (reference "#FLG02") (unit 1)
-        )
-        (path "/05f50450-de9a-44de-96d4-4a146d783d83/d4245743-3101-4aa9-985f-bdd1e5cf8eb9"
-          (reference "#FLG09") (unit 1)
-        )
-      )
-    )
-  )
-  (symbol (lib_id "power:+5V") (at 220.98 87.63 270) (unit 1)
-    (in_bom yes) (on_board yes) (dnp no) (fields_autoplaced)
-    (property "Reference" "#PWR03" (at 217.17 87.63 0)
-      (effects (font (size 1.27 1.27)) hide)
-    )
-    (property "Value" "+5V" (at 224.79 87.63 90)
-      (effects (font (size 1.27 1.27)) (justify left))
-    )
-    (property "Footprint" "" (at 220.98 87.63 0)
-      (effects (font (size 1.27 1.27)) hide)
-    )
-    (property "Datasheet" "" (at 220.98 87.63 0)
-      (effects (font (size 1.27 1.27)) hide)
-    )
-    (pin "1")
-    (instances
-      (project "switched-bandpass-filter"
-        (path "/05f50450-de9a-44de-96d4-4a146d783d83"
-          (reference "#PWR03") (unit 1)
-        )
-        (path "/05f50450-de9a-44de-96d4-4a146d783d83/d4245743-3101-4aa9-985f-bdd1e5cf8eb9"
-          (reference "#PWR09") (unit 1)
-        )
-      )

Commit message: added filter ckt, passes ERC, bumped to v0.2, ready for board layout
Other:
- title: (none) -> switched bandpass filter
Changed lines of the file:
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@@
   (paper "USLetter")
   (title_block
+    (title "switched bandpass filter")
     (date "2023-07-20")
-    (rev "v0.1")
+    (rev "v0.2")
+    (comment 1 "Copyright © 2023 WA7GIL")
   )
   (junction (at 127 85.09) (diameter 0) (color 0 0 0 0)

Commit message: v0.2 passes ERC & DRC except for no solder mask between pads on SOT89
Parts:
- D1, D2, D3, D4: value D -> 1N4148; footprint (none) -> Diode_SMD:D_1210_3225Metric
- Q1, Q2: footprint Package_TO_SOT_THT:TO-92_Inline -> Package_TO_SOT_SMD:SOT-23
- R1, R2, R3, R4: footprint (none) -> Resistor_SMD:R_1210_3225Metric
Changed lines of the file:
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@@
     (in_bom yes) (on_board yes) (dnp no) (fields_autoplaced)
     (property "Reference" "D2" (at 133.35 90.17 0)
-      (effects (font (size 1.27 1.27)))
-    )
-    (property "Value" "D" (at 133.35 92.71 0)
-      (effects (font (size 1.27 1.27)))
-    )
-    (property "Footprint" "" (at 133.35 96.52 0)
+      (effects (font (size 1.27 1.27)) hide)
+    )
+    (property "Value" "1N4148" (at 133.35 92.71 0)
+      (effects (font (size 1.27 1.27)))
+    )
+    (property "Footprint" "Diode_SMD:D_1210_3225Metric" (at 133.35 96.52 0)
       (effects (font (size 1.27 1.27)) hide)
     )
@@
       (effects (font (size 1.27 1.27)) (justify left))
     )
-    (property "Footprint" "Package_TO_SOT_THT:TO-92_Inline" (at 176.53 109.855 0)
+    (property "Footprint" "Package_TO_SOT_SMD:SOT-23" (at 176.53 109.855 0)
       (effects (font (size 1.27 1.27) italic) (justify left) hide)
     )
@@
     (in_bom yes) (on_board yes) (dnp no) (fields_autoplaced)
     (property "Reference" "R4" (at 196.85 93.98 90)
-      (effects (font (size 1.27 1.27)))
+      (effects (font (size 1.27 1.27)) hide)
     )
     (property "Value" "10K" (at 196.85 96.52 90)
       (effects (font (size 1.27 1.27)))
     )
-    (property "Footprint" "" (at 196.85 102.108 90)
+    (property "Footprint" "Resistor_SMD:R_1210_3225Metric" (at 196.85 102.108 90)
       (effects (font (size 1.27 1.27)) hide)
     )
@@
     (in_bom yes) (on_board yes) (dnp no) (fields_autoplaced)
     (property "Reference" "R3" (at 195.58 71.12 90)
-      (effects (font (size 1.27 1.27)))
+      (effects (font (size 1.27 1.27)) hide)
     )
     (property "Value" "10K" (at 195.58 73.66 90)
       (effects (font (size 1.27 1.27)))
     )
-    (property "Footprint" "" (at 195.58 79.248 90)
+    (property "Footprint" "Resistor_SMD:R_1210_3225Metric" (at 195.58 79.248 90)
       (effects (font (size 1.27 1.27)) hide)
     )
@@
     (in_bom yes) (on_board yes) (dnp no) (fields_autoplaced)
     (property "Reference" "R1" (at 153.67 78.74 90)
-      (effects (font (size 1.27 1.27)))
+      (effects (font (size 1.27 1.27)) hide)
     )
     (property "Value" "4.7K" (at 153.67 81.28 90)
       (effects (font (size 1.27 1.27)))
     )
-    (property "Footprint" "" (at 153.67 86.868 90)
+    (property "Footprint" "Resistor_SMD:R_1210_3225Metric" (at 153.67 86.868 90)
       (effects (font (size 1.27 1.27)) hide)
     )
@@
     (in_bom yes) (on_board yes) (dnp no) (fields_autoplaced)
     (property "Reference" "R2" (at 153.67 101.6 90)
-      (effects (font (size 1.27 1.27)))
+      (effects (font (size 1.27 1.27)) hide)
     )
     (property "Value" "4.7K" (at 153.67 104.14 90)
       (effects (font (size 1.27 1.27)))
     )
-    (property "Footprint" "" (at 153.67 106.172 90)
+    (property "Footprint" "Resistor_SMD:R_1210_3225Metric" (at 153.67 106.172 90)
       (effects (font (size 1.27 1.27)) hide)
     )
@@
       (effects (font (size 1.27 1.27)) (justify left))
     )
-    (property "Footprint" "Package_TO_SOT_THT:TO-92_Inline" (at 176.53 86.995 0)
+    (property "Footprint" "Package_TO_SOT_SMD:SOT-23" (at 176.53 86.995 0)
       (effects (font (size 1.27 1.27) italic) (justify left) hide)
     )
@@
     (in_bom yes) (on_board yes) (dnp no) (fields_autoplaced)
     (property "Reference" "D1" (at 133.35 78.74 0)
-      (effects (font (size 1.27 1.27)))
-    )
-    (property "Value" "D" (at 133.35 81.28 0)
-      (effects (font (size 1.27 1.27)))
-    )
-    (property "Footprint" "" (at 133.35 85.09 0)
+      (effects (font (size 1.27 1.27)) hide)
+    )
+    (property "Value" "1N4148" (at 133.35 81.28 0)
+      (effects (font (size 1.27 1.27)))
+    )
+    (property "Footprint" "Diode_SMD:D_1210_3225Metric" (at 133.35 85.09 0)
       (effects (font (size 1.27 1.27)) hide)
     )
@@
     (in_bom yes) (on_board yes) (dnp no) (fields_autoplaced)
     (property "Reference" "D4" (at 133.35 113.03 0)
-      (effects (font (size 1.27 1.27)))
-    )
-    (property "Value" "D" (at 133.35 115.57 0)
-      (effects (font (size 1.27 1.27)))
-    )
-    (property "Footprint" "" (at 133.35 119.38 0)
+      (effects (font (size 1.27 1.27)) hide)
+    )
+    (property "Value" "1N4148" (at 133.35 115.57 0)
+      (effects (font (size 1.27 1.27)))
+    )
+    (property "Footprint" "Diode_SMD:D_1210_3225Metric" (at 133.35 119.38 0)
       (effects (font (size 1.27 1.27)) hide)
     )
@@
     (in_bom yes) (on_board yes) (dnp no) (fields_autoplaced)
     (property "Reference" "D3" (at 133.35 101.6 0)
-      (effects (font (size 1.27 1.27)))
-    )
-    (property "Value" "D" (at 133.35 104.14 0)
-      (effects (font (size 1.27 1.27)))
-    )
-    (property "Footprint" "" (at 133.35 107.95 0)
-      (effects (font (size 1.27 1.27)) hide)
-    )
+      (effects (font (size 1.27 1.27)) hide)
+    )
+    (property "Value" "1N4148" (at 133.35 104.14 0)
+      (effects (font (size 1.27 1.27)))
+    )
+    (property "Footprint" "Diode_SMD:D_1210_3225Metric" (at 133.35 107.95 0)
+      (effects (font (size 1.27 1.27)) hide)
+    )
