File: switched-bandpass-filter.kicad_sch (KiCad schematic)
At the start: 16 parts, among them J1 SMA, J10 F3 out, J11 F4 out, J2 SMA, J3 F4 in, J4 , J5 F3 in, J6 F2 in, J7 F1 in, J8 F1 out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

Commit message: supress display of 1x1 headers for Fx in/out.  Had to supress warnings from DRC as well, since selected component no longer matches what is displayed.  It is intended to be an empty plated through hole.
Parts:
- J4: footprint Connector_PinHeader_2.54mm:PinHeader_1x06_P2.54mm_Vertical -> Connector_PinHeader_2.54mm:PinHeader_1x01_P2.54mm_Vertical
Changed lines of the file:
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@@
       (effects (font (size 1.27 1.27)) hide)
     )
-    (property "Footprint" "Connector_PinHeader_2.54mm:PinHeader_1x06_P2.54mm_Vertical" (at 139.7 33.02 0)
+    (property "Footprint" "Connector_PinHeader_2.54mm:PinHeader_1x01_P2.54mm_Vertical" (at 139.7 33.02 0)
       (effects (font (size 1.27 1.27)) hide)
     )
